File: Hardware/VL6180.brd (EAGLE design)
At the start: 44.5 x 13 mm, 15 parts, among them U1 VL6180, U3 MIC5219 3.3V

Commit message: Boad Layout finished, looking for review
Parts:
- added C4: 0.1uF, SparkFun-Capacitors:0603-CAP
- added FID1, FID2: FIDUCIAL1X2, SparkFun-Aesthetics:FIDUCIAL-1X2
- added LOGO1: SFE_LOGO_NAME_FLAME.1_INCH, SparkFun-Aesthetics:SFE_LOGO_NAME_FLAME_.1
- added LOGO2: OSHW-LOGOS, SparkFun-Aesthetics:OSHW-LOGO-S
- added R5, R6: 4.7k, SparkFun-Resistors:0603
- added U$2: (no value), SparkFun-Aesthetics:SFE_LOGO_FLAME_.1
- R1: value 47K -> 10K
- R2, R3: value (none) -> 4.7k
- moved SJ1 19.2 mm to (22.4, 8.13), turned to 180 degrees
- moved U3 16.4 mm to (5.59, 5.59), turned to 270 degrees
- moved C1 15.7 mm to (10.4, 10.7), turned to 180 degrees
- moved C3 11.6 mm to (17.5, 10.9), turned to 90 degrees
- moved C2 10.6 mm to (10.4, 8.64), turned to 180 degrees
- moved R3 8.98 mm to (15.5, 10.9), turned to 90 degrees
- moved R4 7.10 mm to (8.89, 5.33), turned to 90 degrees
- moved R2 6.42 mm to (13.5, 10.9), turned to 90 degrees
- moved R1 6.27 mm to (10.9, 5.33), turned to 90 degrees
- moved U2 4.58 mm to (18.9, 7.11), turned to 0 degrees
- turned U1 to 90 degrees
Connections:
- new net N$3: R5.2, SJ1.3
- net 2.8V: now also C3.1, U2.8, U3.5
- net GND: now also C3.2, C4.2, U3.2
- net N$2: now also R6.2, SJ1.1; no longer C3.1, U3.5
- net SCL: now also R5.1
- net SDA: now also R6.1
- net VCC: now also C4.1, SJ1.2, U3.1, U3.3
Routing:
- net VCC: track 0.00 -> 28.4 mm, vias 0 -> 3
- net GPIO1: track 0.00 -> 15.0 mm, vias 0 -> 1
- net SCL: track 0.00 -> 13.0 mm
- net SDA: track 0.00 -> 11.5 mm
- net GPIO0: track 0.00 -> 10.9 mm
- net SCL_LV: track 0.00 -> 8.30 mm
- net SDA_LV: track 0.00 -> 7.60 mm, vias 0 -> 2
- net N$2: track 0.00 -> 2.28 mm
- net N$3: track 0.00 -> 2.21 mm
- added copper zone on layer 1, net 2.8V
- added copper zone on layer 1, net GND
- added copper zone on layer 16, net GND
- added copper zone on layer 1, net VCC
Other:
- board text added: "GND"
- board text added: "IO0"
- board text added: "IO1"
- board text added: "Range Finder"
- board text added: "SCL"
- board text added: "SDA"
- board text added: "VCC"
- board text added: "VL6180 TOF"
- board text added: "Vl6180 Time of Flight Range Finder"
- board text added: "v01"
- board text removed: "GPIO0"
