File: Hardware/VL6180.sch (EAGLE design)
At the start: 23 parts, among them U1 VL6180, U3 MIC5219 3.3V

Commit message: added pin 1 designator
Other:
- note added: "v02"
- note removed: "v01"
Changed lines of the file:
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@@
 <plain>
 <text x="166.37" y="11.43" size="2.54" layer="94">Casey Kuhns</text>
-<text x="238.76" y="6.35" size="2.54" layer="94">v01</text>
+<text x="238.76" y="6.35" size="2.54" layer="94">v02</text>
 </plain>
 <instances>
